File: Mirley_ESP8266.sch (EAGLE design)
At the start: 83 parts, among them J1 61301611121, J10 61300511121, J2 61301611121, J3 61300211121, J6 61300811121, J8 61300811121, T1 BC817U, T10 BC817U, T11 BC817U, T12 BC817U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

Commit message: pierwsza wersja na jedenj plytce, niedokonczona
Parts:
- removed R59, R60: 10K, rcl:R-EU_R0805
- added JP1: (no value), pinhead:PINHD-2X2
- R10, R27, R28, R29, R3, R30, R31, R32, R33, R34, R4, R5, R6, R7, R8, R9: device rcl:R-EU_R0805 -> rcl:R-EU_R0603
Connections:
- removed net ACD0: ESP_2.ADC
- removed net ADC0: J10.4, R54.1, R54.2, R55.2
- new net ADC: ESP_2.ADC, R54.1, R55.2
- new net N$10: J10.4, R54.2
- new net N$5: U$1.3V3, U$1.VCC
- net +3V3: now also JP1.1, JP1.2, JP1.3, JP1.4; no longer R59.1, R60.1
- net ENABLE: no longer R60.2
- net RESET: no longer R59.2
Other:
- moved on the sheet: J1, J2

Commit message: pytlka programoatora w 50% narysowana
Parts:
- removed C1: 100nF, rcl:C-EUC0805K
- removed C2, C4: 10uF, rcl:C-EUC0805K
- removed G1: (no value), infineon:IFX1117ME_V33
- removed J3: 61300211121, Headers:61300211121
- removed JP1: (no value), pinhead:PINHD-2X2
- removed R1, R2: 10K, rcl:R-EU_R0805
- removed R57: 47K, rcl:R-EU_R0805
- removed T1: BC817U, transistor:BC817U
- removed U$1: USB-SERIAL-CH340, diy-modules:USB-SERIAL-CH340
- removed U$4: WIRELESS-WIFI-ESP-01, diy-modules:WIRELESS-WIFI-ESP-01
Connections:
- removed net DTR: R1.1, T1G$2.E, U$1.DTR
- removed net N$1: R2.1, T1G$2.B
- removed net N$2: R1.2, T1G$1.B
- removed net N$5: U$1.3V3, U$1.VCC
- removed net RTS: R2.2, T1G$1.E, U$1.RTS
- net +3V3: now also J2.6, J2.7; no longer C4.1, G1.Q_1, G1.Q_2, JP1.1, JP1.2, JP1.3, JP1.4, R57.2, U$4.VCC
- net +5V: no longer C1.1, C2.1, G1.I, U$1.PLUS
- net D+: no longer U$1.D+
- net D-: no longer U$1.D-
- net ENABLE: no longer U$4.RST
- net GND: no longer C1.2, C2.2, C4.2, G1.GND, U$1.GND, U$1.MINUS, U$4.GND
- net GPIO0: now also J2.10; no longer T1G$2.C, U$4.GPIO0
- net GPIO16: no longer J3.2
- net GPIO2: no longer U$4.GPIO2
- net RESET: no longer J3.1, T1G$1.C, U$4.CH_PD
- net RXD: no longer U$1.TXD, U$4.URXD
- net TXD: no longer R57.1, U$1.RXD, U$4.UTXD
Other:
- note removed: "ESP8266-01"
- note removed: "USB -> UART"
- moved on the sheet: C3

Commit message: programator zrobiony
Parts:
- removed ESP_2: ESP8266-12-WITH-ADAPTER, esp8266_with_adapter:ESP8266-12-WITH-ADAPTER
- removed R53, R56: 10K, rcl:R-EU_R0805
- removed S1: (no value), switch-dil:DIP02YL
- added ESP_1: ESP8266-12-WITH-ADAPTER, esp8266_with_adapter:ESP8266-12-WITH-ADAPTER
- added R1, R2: 10K, rcl:R-EU_R0805
- added S2: (no value), switch-dil:DIP02YL
Connections:
- net +3V3: now also ESP_1.VCC3V3, R1.1, R2.1; no longer ESP_2.VCC3V3, R53.1, R56.1
- net ADC: now also ESP_1.ADC; no longer ESP_2.ADC
- net ENABLE: now also ESP_1.CH_PD, R2.2; no longer ESP_2.CH_PD, R56.2
- net GND: now also ESP_1.GND; no longer ESP_2.GND
- net GPIO0: now also ESP_1.GPIO0; no longer ESP_2.GPIO0
- net GPIO1: now also S2.1; no longer S1.1
- net GPIO10: now also ESP_1.GPIO10; no longer ESP_2.GPIO10
- net GPIO11: now also ESP_1.CS0; no longer ESP_2.CS0
- net GPIO12: now also ESP_1.GPIO12; no longer ESP_2.GPIO12
- net GPIO13: now also ESP_1.GPIO13; no longer ESP_2.GPIO13
- net GPIO14: now also ESP_1.GPIO14; no longer ESP_2.GPIO14
- net GPIO15: now also ESP_1.GPIO15; no longer ESP_2.GPIO15
- net GPIO16: now also ESP_1.GPIO16; no longer ESP_2.GPIO16
- net GPIO2: now also ESP_1.GPIO2; no longer ESP_2.GPIO2
- net GPIO3: now also S2.2; no longer S1.2
- net GPIO4: now also ESP_1.GPIO4; no longer ESP_2.GPIO4
- net GPIO5: now also ESP_1.GPIO5; no longer ESP_2.GPIO5
- net GPIO6: now also ESP_1.SCLK; no longer ESP_2.SCLK
- net GPIO7: now also ESP_1.MISO; no longer ESP_2.MISO
- net GPIO8: now also ESP_1.MOSI; no longer ESP_2.MOSI
- net GPIO9: now also ESP_1.GPIO9; no longer ESP_2.GPIO9
- net RESET: now also ESP_1.REST, R1.2; no longer ESP_2.REST, R53.2
- net RXD: now also ESP_1.RXD, S2.3; no longer ESP_2.RXD, S1.3
- net TXD: now also ESP_1.TXD, S2.4; no longer ESP_2.TXD, S1.4
Other:
- note removed: "ESP8266-12 ESP8266-07 ESP8266-01"

Commit message: usb-uart skonczone, druga skonczona w 50%
Parts:
- removed J10: 61300511121, Headers:61300511121
- removed J6: 61300811121, Headers:61300811121
- added JP1: (no value), pinhead:PINHD-2X8
- added JP2: (no value), pinhead:PINHD-1X2
- added JP3: (no value), pinhead:PINHD-1X3
- J8: value 61300811121 -> (none); device Headers:61300811121 -> pinhead:PINHD-2X8
Connections:
- removed net LED_A4]: J1.12
- removed net N$10: J10.4, R54.2
- removed net N$9: J6.2, R44.1, T7G$2.C
- new net N$1: JP1.3, JP1.4, R44.1, T7G$2.C
- new net N$2: JP3.2, R54.2
- net +3V3: now also J2.5; no longer J2.7
- net ENABLE: now also JP3.1; no longer J10.2
- net GND: now also J2.7; no longer J10.3, J2.9
- net GPIO0: now also J2.9; no longer J2.10
- net GPIO1: now also S2.2; no longer S2.1
- net GPIO16: now also JP2.1, JP2.2; no longer J10.5
- net GPIO3: now also S2.1; no longer S2.2
- net LED_A1: now also JP1.11, JP1.12; no longer J6.6
- net LED_A2: now also JP1.10, JP1.9; no longer J6.5
- net LED_A3: now also JP1.7, JP1.8; no longer J6.4
- net LED_A4: now also J1.12, JP1.5, JP1.6; no longer J6.3
- net LL1: now also J8.2
- net LL2: now also J8.3, J8.4; no longer J8.2
- net LL3: now also J8.10, J8.9; no longer J8.5
- net LL4: now also J8.11, J8.12; no longer J8.6
- net LL5: now also J8.13, J8.14; no longer J8.7
- net LL6: now also J8.15, J8.16; no longer J8.8
- net LL7: now also JP1.15, JP1.16; no longer J6.8
- net LL8: now also JP1.13, JP1.14; no longer J6.7
- net N$3: now also JP1.1, JP1.2; no longer J6.1
- net RESET: now also J2.10, JP3.3; no longer J10.1
- net RXD: now also ESP_1.TXD, J2.4; no longer ESP_1.RXD, J2.5
- net SCL: now also J8.7, J8.8; no longer J8.4
- net SDA: now also J8.5, J8.6; no longer J8.3
- net TXD: now also ESP_1.RXD, J2.3; no longer ESP_1.TXD, J2.4
Other:
- moved on the sheet: R51, R52, R54, R55

Commit message: pierwsza docelowa wersja
Connections:
- net GPIO10: now also T11G$1.E; no longer T14G$2.E
- net GPIO11: now also T10G$1.E; no longer T14G$1.E
- net GPIO14: now also T12G$1.E; no longer T12G$2.E
- net GPIO15: now also JP2.1, JP2.2, R51.2
- net GPIO16: now also T12G$2.E; no longer JP2.1, JP2.2, R51.2, T12G$1.E
- net GPIO6: now also T14G$1.E; no longer T10G$1.E
- net GPIO8: now also T14G$2.E; no longer T11G$1.E
- net LED_A3: now also T12G$1.C; no longer T12G$2.C
- net LED_A4: now also T12G$2.C; no longer T12G$1.C
- net LL3: now also T14G$1.C; no longer T10G$1.C
- net LL5: now also T14G$2.C; no longer T11G$1.C
- net LL7: now also T11G$1.C; no longer T14G$2.C
- net LL8: now also T10G$1.C; no longer T14G$1.C
- net N$14: now also T12G$2.B; no longer T12G$1.B
- net N$15: now also T12G$1.B; no longer T12G$2.B
- net N$20: now also T14G$1.B; no longer T10G$1.B
- net N$27: now also T10G$1.B; no longer T14G$1.B
- net N$28: now also T14G$2.B; no longer T11G$1.B
- net N$31: now also T11G$1.B; no longer T14G$2.B
Other:
- moved on the sheet: T10G$1, T11G$1, T12G$1, T12G$2, T14G$1, T14G$2
