File: Mirley_USB-UART.sch (EAGLE design)
At the start: 34 parts, among them J1 61301611121, J2 61301611121, J4 62000311121, J7 62000811121, T1 BC817U, T2 BC817U, T3 BC817U

Commit message: programator zrobiony
Changed lines of the file:
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@@
 <part name="+3V26" library="supply1" library_urn="urn:adsk.eagle:library:371" deviceset="+3V3" device=""/>
 <part name="+3V27" library="supply1" library_urn="urn:adsk.eagle:library:371" deviceset="+3V3" device=""/>
-<part name="JP2" library="pinhead" library_urn="urn:adsk.eagle:library:13445724" deviceset="PINHD-2X4" device="" package3d_urn="urn:adsk.eagle:package:22461/2"/>
+<part name="JP2" library="pinhead" library_urn="urn:adsk.eagle:library:13445724" deviceset="PINHD-2X4" device="" package3d_urn="urn:adsk.eagle:package:15331965/1"/>
 </parts>
 <sheets>
@@
 <wire x1="121.92" y1="43.18" x2="129.54" y2="43.18" width="0.1524" layer="91"/>
 <junction x="121.92" y="43.18"/>
+<label x="111.76" y="66.04" size="1.778" layer="95"/>
 </segment>
 </net>
@@
 <wire x1="121.92" y1="40.64" x2="129.54" y2="40.64" width="0.1524" layer="91"/>
 <junction x="121.92" y="40.64"/>
+<label x="111.76" y="48.26" size="1.778" layer="95"/>
 </segment>
 </net>
@@
 <wire x1="121.92" y1="38.1" x2="129.54" y2="38.1" width="0.1524" layer="91"/>
 <junction x="121.92" y="38.1"/>
+<label x="109.22" y="30.48" size="1.778" layer="95"/>
 </segment>
 </net>
@@
 <wire x1="121.92" y1="35.56" x2="129.54" y2="35.56" width="0.1524" layer="91"/>
 <junction x="121.92" y="35.56"/>
-</segment>
-</net>
+<label x="111.76" y="12.7" size="1.778" layer="95"/>
+</segment>
+</net>

Commit message: usb-uart skonczone, druga skonczona w 50%
Connections:
- net +3V3: now also J2.5; no longer J2.7
- net GND: now also J2.7; no longer J2.9
- net GPIO0: now also J2.9; no longer J2.10
- net GPIO1: now also S1.2; no longer S1.1
- net GPIO3: now also S1.1; no longer S1.2
- net RESET: now also J2.10
- net RXD: now also J2.4, U$1.RXD, U$4.UTXD; no longer J2.5, U$1.TXD, U$4.URXD
- net TXD: now also J2.3, U$1.TXD, U$4.URXD; no longer J2.4, U$1.RXD, U$4.UTXD
Changed lines of the file:
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@@
 <drawing>
 <settings>
-<setting alwaysvectorfont="no"/>
+<setting alwaysvectorfont="yes"/>
 <setting verticaltext="up"/>
 </settings>
@@
 <attribute name="VALUE" x="182.88" y="111.76" size="1.778" layer="96" rot="MR180"/>
 </instance>
-<instance part="GND1" gate="1" x="180.34" y="132.08" smashed="yes" rot="MR0">
-<attribute name="VALUE" x="182.88" y="129.54" size="1.778" layer="96" rot="MR0"/>
+<instance part="GND1" gate="1" x="180.34" y="134.62" smashed="yes" rot="MR0">
+<attribute name="VALUE" x="182.88" y="132.08" size="1.778" layer="96" rot="MR0"/>
 </instance>
 <instance part="GND2" gate="1" x="27.94" y="86.36" smashed="yes" rot="MR0">
@@
 <attribute name="VALUE" x="139.7" y="88.9" size="1.778" layer="96" rot="R180"/>
 </instance>
-<instance part="+3V23" gate="G$1" x="187.96" y="132.08" smashed="yes" rot="R180">
-<attribute name="VALUE" x="185.42" y="129.54" size="1.778" layer="96"/>
+<instance part="+3V23" gate="G$1" x="187.96" y="134.62" smashed="yes" rot="R180">
+<attribute name="VALUE" x="185.42" y="132.08" size="1.778" layer="96"/>
 </instance>
 <instance part="J4" gate="G$1" x="78.74" y="83.82" smashed="yes" rot="R90">
@@
 <segment>
 <pinref part="GND1" gate="1" pin="GND"/>
-<wire x1="180.34" y1="134.62" x2="180.34" y2="137.16" width="0.1524" layer="91"/>
-<pinref part="J2" gate="G$1" pin="9"/>
-<wire x1="170.18" y1="134.62" x2="172.72" y2="134.62" width="0.1524" layer="91"/>
-<wire x1="172.72" y1="134.62" x2="172.72" y2="137.16" width="0.1524" layer="91"/>
+<pinref part="J2" gate="G$1" pin="7"/>
+<wire x1="170.18" y1="139.7" x2="175.26" y2="139.7" width="0.1524" layer="91"/>
+<wire x1="175.26" y1="139.7" x2="180.34" y2="139.7" width="0.1524" layer="91"/>
+<wire x1="180.34" y1="139.7" x2="180.34" y2="137.16" width="0.1524" layer="91"/>
 <pinref part="J2" gate="G$1" pin="8"/>
-<wire x1="172.72" y1="137.16" x2="170.18" y2="137.16" width="0.1524" layer="91"/>
-<wire x1="172.72" y1="137.16" x2="180.34" y2="137.16" width="0.1524" layer="91"/>
-<junction x="172.72" y="137.16"/>
+<wire x1="170.18" y1="137.16" x2="175.26" y2="137.16" width="0.1524" layer="91"/>
+<wire x1="175.26" y1="137.16" x2="175.26" y2="139.7" width="0.1524" layer="91"/>
+<junction x="175.26" y="139.7"/>
 </segment>
 <segment>
@@
 <net name="TXD" class="0">
 <segment>
-<pinref part="U$1" gate="G$1" pin="RXD"/>
-<wire x1="73.66" y1="101.6" x2="76.2" y2="101.6" width="0.1524" layer="91"/>
-<label x="76.2" y="101.6" size="1.27" layer="95" xref="yes"/>
-</segment>
-<segment>
-<pinref part="J2" gate="G$1" pin="4"/>
-<wire x1="170.18" y1="147.32" x2="180.34" y2="147.32" width="0.1524" layer="91"/>
-<label x="180.34" y="147.32" size="1.27" layer="95" xref="yes"/>
+<label x="180.34" y="149.86" size="1.27" layer="95" xref="yes"/>
+<pinref part="J2" gate="G$1" pin="3"/>
+<wire x1="170.18" y1="149.86" x2="180.34" y2="149.86" width="0.1524" layer="91"/>
 </segment>
 <segment>
@@
 <label x="162.56" y="73.66" size="1.27" layer="95" rot="R270" xref="yes"/>
 <pinref part="J7" gate="G$1" pin="6"/>
+</segment>
+<segment>
+<pinref part="U$1" gate="G$1" pin="TXD"/>
+<wire x1="73.66" y1="99.06" x2="76.2" y2="99.06" width="0.1524" layer="91"/>
+<label x="76.2" y="99.06" size="1.27" layer="95" xref="yes"/>
 </segment>
 </net>
@@
 <segment>
 <pinref part="J2" gate="G$1" pin="14"/>
-<wire x1="170.18" y1="121.92" x2="177.8" y2="121.92" width="0.1524" layer="91"/>
+<wire x1="170.18" y1="121.92" x2="172.72" y2="121.92" width="0.1524" layer="91"/>
 <label x="177.8" y="121.92" size="1.27" layer="95" xref="yes"/>
+<pinref part="J2" gate="G$1" pin="10"/>
+<wire x1="172.72" y1="121.92" x2="177.8" y2="121.92" width="0.1524" layer="91"/>
+<wire x1="170.18" y1="132.08" x2="172.72" y2="132.08" width="0.1524" layer="91"/>
+<wire x1="172.72" y1="132.08" x2="172.72" y2="121.92" width="0.1524" layer="91"/>
+<junction x="172.72" y="121.92"/>
 </segment>
 <segment>
@@
 </segment>
 <segment>
-<pinref part="J2" gate="G$1" pin="10"/>
-<wire x1="170.18" y1="132.08" x2="172.72" y2="132.08" width="0.1524" layer="91"/>
-<wire x1="172.72" y1="132.08" x2="172.72" y2="126.492" width="0.1524" layer="91"/>
-<wire x1="172.72" y1="126.492" x2="177.292" y2="126.492" width="0.1524" layer="91"/>
-<label x="177.292" y="126.492" size="1.27" layer="95" xref="yes"/>
+<wire x1="175.26" y1="134.62" x2="175.26" y2="129.032" width="0.1524" layer="91"/>
+<wire x1="175.26" y1="129.032" x2="177.292" y2="129.032" width="0.1524" layer="91"/>
+<label x="177.292" y="129.032" size="1.27" layer="95" xref="yes"/>
+<pinref part="J2" gate="G$1" pin="9"/>
+<wire x1="170.18" y1="134.62" x2="175.26" y2="134.62" width="0.1524" layer="91"/>
 </segment>
 <segment>
@@
 </segment>
 <segment>
-<pinref part="J2" gate="G$1" pin="7"/>
-<wire x1="170.18" y1="139.7" x2="180.34" y2="139.7" width="0.1524" layer="91"/>
-<wire x1="180.34" y1="139.7" x2="180.34" y2="142.24" width="0.1524" layer="91"/>
 <pinref part="J2" gate="G$1" pin="6"/>
 <wire x1="180.34" y1="142.24" x2="170.18" y2="142.24" width="0.1524" layer="91"/>
-<wire x1="180.34" y1="139.7" x2="187.96" y2="139.7" width="0.1524" layer="91"/>
-<wire x1="187.96" y1="139.7" x2="187.96" y2="134.62" width="0.1524" layer="91"/>
-<junction x="180.34" y="139.7"/>
+<wire x1="180.34" y1="142.24" x2="187.96" y2="142.24" width="0.1524" layer="91"/>
+<wire x1="187.96" y1="142.24" x2="187.96" y2="137.16" width="0.1524" layer="91"/>
 <pinref part="+3V23" gate="G$1" pin="+3V3"/>
+<pinref part="J2" gate="G$1" pin="5"/>
+<wire x1="170.18" y1="144.78" x2="180.34" y2="144.78" width="0.1524" layer="91"/>
+<wire x1="180.34" y1="144.78" x2="180.34" y2="142.24" width="0.1524" layer="91"/>
+<junction x="180.34" y="142.24"/>
 </segment>
 <segment>
@@
 <net name="RXD" class="0">
 <segment>
-<pinref part="U$1" gate="G$1" pin="TXD"/>
-<wire x1="73.66" y1="99.06" x2="76.2" y2="99.06" width="0.1524" layer="91"/>
-<label x="76.2" y="99.06" size="1.27" layer="95" xref="yes"/>
-</segment>
-<segment>
-<pinref part="J2" gate="G$1" pin="5"/>
-<wire x1="170.18" y1="144.78" x2="180.34" y2="144.78" width="0.1524" layer="91"/>
-<label x="180.34" y="144.78" size="1.27" layer="95" xref="yes"/>
+<label x="180.34" y="147.32" size="1.27" layer="95" xref="yes"/>
+<pinref part="J2" gate="G$1" pin="4"/>
+<wire x1="170.18" y1="147.32" x2="180.34" y2="147.32" width="0.1524" layer="91"/>
 </segment>
 <segment>
@@
 <label x="165.1" y="73.66" size="1.27" layer="95" rot="R270" xref="yes"/>
 <pinref part="J7" gate="G$1" pin="5"/>
+</segment>
+<segment>
+<pinref part="U$1" gate="G$1" pin="RXD"/>
+<wire x1="73.66" y1="101.6" x2="76.2" y2="101.6" width="0.1524" layer="91"/>
+<label x="76.2" y="101.6" size="1.27" layer="95" xref="yes"/>
 </segment>
 </net>
@@
 <net name="TXD" class="0">
 <segment>
-<pinref part="U$4" gate="G$1" pin="UTXD"/>
-<wire x1="78.74" y1="132.08" x2="66.04" y2="132.08" width="0.1524" layer="91"/>
-<label x="66.04" y="132.08" size="1.4224" layer="95" rot="R180" xref="yes"/>
-</segment>
-<segment>
 <pinref part="S1" gate="1" pin="4"/>
 <wire x1="175.26" y1="137.16" x2="175.26" y2="139.7" width="0.1524" layer="91"/>
@@
 <pinref part="R57" gate="G$1" pin="1"/>
 </segment>
-</net>
-<net name="RXD" class="0">
 <segment>
 <pinref part="U$4" gate="G$1" pin="URXD"/>
@@
 <label x="66.04" y="119.38" size="1.4224" layer="95" rot="R180" xref="yes"/>
 </segment>
+</net>
+<net name="RXD" class="0">
 <segment>
 <pinref part="S1" gate="1" pin="3"/>
@@
 <wire x1="177.8" y1="139.7" x2="185.42" y2="139.7" width="0.1524" layer="91"/>
 <label x="185.42" y="139.7" size="1.4224" layer="95" xref="yes"/>
+</segment>
+<segment>
+<pinref part="U$4" gate="G$1" pin="UTXD"/>
+<wire x1="78.74" y1="132.08" x2="66.04" y2="132.08" width="0.1524" layer="91"/>
+<label x="66.04" y="132.08" size="1.4224" layer="95" rot="R180" xref="yes"/>
 </segment>
 </net>
@@
 <net name="GPIO1" class="0">
 <segment>
-<pinref part="S1" gate="1" pin="1"/>
-<wire x1="175.26" y1="121.92" x2="175.26" y2="119.38" width="0.1524" layer="91"/>
-<wire x1="175.26" y1="119.38" x2="162.56" y2="119.38" width="0.1524" layer="91"/>
-<label x="162.56" y="119.38" size="1.4224" layer="95" rot="R180" xref="yes"/>
-</segment>
-<segment>
 <pinref part="R64" gate="G$1" pin="1"/>
 <pinref part="T2" gate="G$2" pin="E"/>
@@
 <label x="38.1" y="48.26" size="1.27" layer="95" rot="R180" xref="yes"/>
 </segment>
-</net>
-<net name="GPIO3" class="0">
 <segment>
 <pinref part="S1" gate="1" pin="2"/>
@@
 <label x="185.42" y="119.38" size="1.4224" layer="95" xref="yes"/>
 </segment>
+</net>
+<net name="GPIO3" class="0">
 <segment>
 <pinref part="R66" gate="G$1" pin="1"/>
@@
 <label x="38.1" y="12.7" size="1.27" layer="95" rot="R180" xref="yes"/>
 </segment>
-</net>
+<segment>
+<pinref part="S1" gate="1" pin="1"/>
+<wire x1="175.26" y1="121.92" x2="175.26" y2="119.38" width="0.1524" layer="91"/>
+<wire x1="175.26" y1="119.38" x2="162.56" y2="119.38" width="0.1524" layer="91"/>
+<label x="162.56" y="119.38" size="1.4224" layer="95" rot="R180" xref="yes"/>
+</segment>
+</net>

Commit message: powiekszonyy odstepy miedzy sciezkami
Parts:
- removed J4: 62000311121, Headers:62000311121
- removed J7: 62000811121, Headers:62000811121
- added JP3: (no value), pinhead:PINHD-1X8
- added JP4: (no value), pinhead:PINHD-1X3
Connections:
- net +3V3: now also JP3.1; no longer J7.8
- net DTR: now also JP3.8; no longer J7.1
- net GND: now also JP3.2; no longer J7.7
- net GPIO0: now also JP3.5; no longer J7.4
- net N$11: now also JP4.2; no longer J4.2
- net N$13: now also JP4.1; no longer J4.3
- net N$5: now also JP4.3; no longer J4.1
- net RESET: now also JP3.6; no longer J7.3
- net RTS: now also JP3.7; no longer J7.2
- net RXD: now also JP3.4; no longer J7.5
- net TXD: now also JP3.3; no longer J7.6
Changed lines of the file:
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@@
 <part name="+3V22" library="supply1" library_urn="urn:adsk.eagle:library:371" deviceset="+3V3" device=""/>
 <part name="+3V23" library="supply1" library_urn="urn:adsk.eagle:library:371" deviceset="+3V3" device=""/>
-<part name="J4" library="Headers" library_urn="urn:adsk.eagle:library:13525965" deviceset="62000311121" device="" package3d_urn="urn:adsk.eagle:package:15328753/1"/>
 <part name="+3V24" library="supply1" library_urn="urn:adsk.eagle:library:371" deviceset="+3V3" device=""/>
 <part name="GND9" library="supply1" library_urn="urn:adsk.eagle:library:371" deviceset="GND" device="">
 <attribute name="SPICEPREFIX" value="G"/>
-</part>
-<part name="J7" library="Headers" library_urn="urn:adsk.eagle:library:13525965" deviceset="62000811121" device="" package3d_urn="urn:adsk.eagle:package:15328572/1">
-<attribute name="SPICEPREFIX" value="X"/>
 </part>
 <part name="R58" library="rcl" library_urn="urn:adsk.eagle:library:13439567" deviceset="R-EU_" device="R0805" package3d_urn="urn:adsk.eagle:package:23553/2" value="10K"/>
@@
 <part name="+3V27" library="supply1" library_urn="urn:adsk.eagle:library:371" deviceset="+3V3" device=""/>
 <part name="JP2" library="pinhead" library_urn="urn:adsk.eagle:library:13445724" deviceset="PINHD-2X4" device="" package3d_urn="urn:adsk.eagle:package:15331965/1"/>
+<part name="JP3" library="pinhead" library_urn="urn:adsk.eagle:library:13445724" deviceset="PINHD-1X8" device="" package3d_urn="urn:adsk.eagle:package:22409/2"/>
+<part name="JP4" library="pinhead" library_urn="urn:adsk.eagle:library:13445724" deviceset="PINHD-1X3" device="" package3d_urn="urn:adsk.eagle:package:22458/2"/>
 </parts>
 <sheets>
@@
 <attribute name="VALUE" x="185.42" y="132.08" size="1.778" layer="96"/>
 </instance>
-<instance part="J4" gate="G$1" x="78.74" y="83.82" smashed="yes" rot="R90">
-<attribute name="NAME" x="73.152" y="81.534" size="1.778" layer="95" rot="R90"/>
-</instance>
 <instance part="+3V24" gate="G$1" x="149.86" y="86.36" smashed="yes">
 <attribute name="VALUE" x="152.4" y="88.9" size="1.778" layer="96" rot="R180"/>
@@
 <attribute name="VALUE" x="160.02" y="63.5" size="1.778" layer="96" rot="MR0"/>
 </instance>
-<instance part="J7" gate="G$1" x="167.64" y="86.36" smashed="yes" rot="R270">
-<attribute name="NAME" x="180.848" y="86.36" size="1.778" layer="95" rot="R270"/>
+<instance part="JP3" gate="A" x="167.64" y="86.36" smashed="yes" rot="R90">
+<attribute name="NAME" x="154.305" y="80.01" size="1.778" layer="95" rot="R90"/>
+<attribute name="VALUE" x="180.34" y="80.01" size="1.778" layer="96" rot="R90"/>
+</instance>
+<instance part="JP4" gate="A" x="78.74" y="86.36" smashed="yes" rot="R270">
+<attribute name="NAME" x="84.455" y="92.71" size="1.778" layer="95" rot="R270"/>
+<attribute name="VALUE" x="71.12" y="92.71" size="1.778" layer="96" rot="R270"/>
 </instance>
 </instances>
@@
 </segment>
 <segment>
-<pinref part="J7" gate="G$1" pin="7"/>
-<wire x1="160.02" y1="81.28" x2="160.02" y2="73.66" width="0.1524" layer="91"/>
 <wire x1="160.02" y1="73.66" x2="157.48" y2="73.66" width="0.1524" layer="91"/>
 <pinref part="GND9" gate="1" pin="GND"/>
 <wire x1="157.48" y1="73.66" x2="157.48" y2="68.58" width="0.1524" layer="91"/>
+<pinref part="JP3" gate="A" pin="2"/>
+<wire x1="160.02" y1="73.66" x2="160.02" y2="83.82" width="0.1524" layer="91"/>
 </segment>
 </net>
@@
 </segment>
 <segment>
-<wire x1="162.56" y1="81.28" x2="162.56" y2="73.66" width="0.1524" layer="91"/>
 <label x="162.56" y="73.66" size="1.27" layer="95" rot="R270" xref="yes"/>
-<pinref part="J7" gate="G$1" pin="6"/>
+<pinref part="JP3" gate="A" pin="3"/>
+<wire x1="162.56" y1="73.66" x2="162.56" y2="83.82" width="0.1524" layer="91"/>
 </segment>
 <segment>
@@
 </segment>
 <segment>
-<pinref part="J7" gate="G$1" pin="2"/>
-<wire x1="172.72" y1="81.28" x2="172.72" y2="73.66" width="0.1524" layer="91"/>
+<pinref part="JP3" gate="A" pin="7"/>
+<wire x1="172.72" y1="83.82" x2="172.72" y2="73.66" width="0.1524" layer="91"/>
 <label x="172.72" y="73.66" size="1.27" layer="95" rot="R270" xref="yes"/>
 </segment>
@@
 </segment>
 <segment>
-<pinref part="J7" gate="G$1" pin="1"/>
-<wire x1="175.26" y1="81.28" x2="175.26" y2="73.66" width="0.1524" layer="91"/>
+<wire x1="175.26" y1="83.82" x2="175.26" y2="73.66" width="0.1524" layer="91"/>
 <label x="175.26" y="73.66" size="1.27" layer="95" rot="R270" xref="yes"/>
+<pinref part="JP3" gate="A" pin="8"/>
 </segment>
 </net>
@@
 </segment>
 <segment>
-<wire x1="170.18" y1="81.28" x2="170.18" y2="73.66" width="0.1524" layer="91"/>
+<pinref part="JP3" gate="A" pin="6"/>
+<wire x1="170.18" y1="83.82" x2="170.18" y2="73.66" width="0.1524" layer="91"/>
 <label x="170.18" y="73.66" size="1.27" layer="95" rot="R270" xref="yes"/>
-<pinref part="J7" gate="G$1" pin="3"/>
 </segment>
 </net>
@@
 </segment>
 <segment>
-<wire x1="167.64" y1="81.28" x2="167.64" y2="73.66" width="0.1524" layer="91"/>
 <label x="167.64" y="73.66" size="1.27" layer="95" rot="R270" xref="yes"/>
-<pinref part="J7" gate="G$1" pin="4"/>
+<pinref part="JP3" gate="A" pin="5"/>
+<wire x1="167.64" y1="73.66" x2="167.64" y2="83.82" width="0.1524" layer="91"/>
 </segment>
 </net>
@@
 </segment>
 <segment>
-<wire x1="157.48" y1="81.28" x2="157.48" y2="76.2" width="0.1524" layer="91"/>
 <wire x1="157.48" y1="76.2" x2="149.86" y2="76.2" width="0.1524" layer="91"/>
 <pinref part="+3V24" gate="G$1" pin="+3V3"/>
 <wire x1="149.86" y1="83.82" x2="149.86" y2="76.2" width="0.1524" layer="91"/>
-<pinref part="J7" gate="G$1" pin="8"/>
+<pinref part="JP3" gate="A" pin="1"/>
+<wire x1="157.48" y1="76.2" x2="157.48" y2="83.82" width="0.1524" layer="91"/>
 </segment>
 </net>
@@
 </segment>
 <segment>
-<wire x1="165.1" y1="81.28" x2="165.1" y2="73.66" width="0.1524" layer="91"/>
 <label x="165.1" y="73.66" size="1.27" layer="95" rot="R270" xref="yes"/>
-<pinref part="J7" gate="G$1" pin="5"/>
+<pinref part="JP3" gate="A" pin="4"/>
+<wire x1="165.1" y1="73.66" x2="165.1" y2="83.82" width="0.1524" layer="91"/>
 </segment>
 <segment>
@@
 <net name="N$5" class="0">
 <segment>
-<pinref part="J4" gate="G$1" pin="1"/>
 <pinref part="U$1" gate="G$1" pin="5V"/>
 <wire x1="76.2" y1="88.9" x2="76.2" y2="91.44" width="0.1524" layer="91"/>
 <wire x1="76.2" y1="91.44" x2="73.66" y2="91.44" width="0.1524" layer="91"/>
+<pinref part="JP4" gate="A" pin="3"/>
 </segment>
 </net>
@@
 <pinref part="U$1" gate="G$1" pin="VCC"/>
 <wire x1="73.66" y1="93.98" x2="78.74" y2="93.98" width="0.1524" layer="91"/>
-<pinref part="J4" gate="G$1" pin="2"/>
 <wire x1="78.74" y1="93.98" x2="78.74" y2="88.9" width="0.1524" layer="91"/>
+<pinref part="JP4" gate="A" pin="2"/>
 </segment>
 </net>
@@
 <segment>
 <pinref part="U$1" gate="G$1" pin="3V3"/>
-<pinref part="J4" gate="G$1" pin="3"/>
 <wire x1="73.66" y1="96.52" x2="81.28" y2="96.52" width="0.1524" layer="91"/>
 <wire x1="81.28" y1="96.52" x2="81.28" y2="88.9" width="0.1524" layer="91"/>
-</segment>
-</net>
+<pinref part="JP4" gate="A" pin="1"/>
+</segment>
+</net>
