File: Mirley_USB-UART.brd (EAGLE design)
At the start: 52 x 69.4 mm, 34 parts, among them J1 61301611121, J2 61301611121, J4 62000311121, J7 62000811121, T1 BC817U, T2 BC817U, T3 BC817U

Commit message: pytlka programoatora w 50% narysowana
Parts:
- moved S1 64.6 mm to (43.1, 59.5)
- moved C3 49.6 mm to (-11.2, 22.4)
- moved JP1 44.1 mm to (5.10, 7.08)
- moved G1 33.8 mm to (26.6, 12.7), turned to 180 degrees
- moved R56 31.4 mm to (-19.9, 56.0), turned to 180 degrees
- moved C4 26.5 mm to (18.1, 16.4)
- moved T1 22.5 mm to (42.7, 24.3), turned to 0 degrees
- moved R1 16.0 mm to (42.8, 20.9), turned to 180 degrees
- moved C1 15.5 mm to (21.2, 9.27)
- moved C2 15.2 mm to (19.0, 9.29)
- moved JP2 15.1 mm to (11.7, 60.2)
- moved R2 13.8 mm to (42.9, 27.8), turned to 180 degrees
- moved U$4 13.2 mm to (26.2, 56.0), turned to 90 degrees
- moved J4 6.11 mm to (43.7, 9.47)
- moved J7 1.40 mm to (25.8, 27.7)
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Routing:
- net +3V3: track 0.00 -> 152.1 mm, vias 0 -> 4
- net GND: track 0.00 -> 103.5 mm, vias 0 -> 4
- net +5V: track 0.00 -> 94.7 mm, vias 0 -> 4
- net DTR: track 0.00 -> 57.1 mm, vias 0 -> 4
- net RTS: track 0.00 -> 45.1 mm, vias 0 -> 2
- net RESET: track 0.00 -> 39.0 mm, vias 0 -> 2
- net RXD: track 0.00 -> 38.4 mm, vias 0 -> 4
- net TXD: track 0.00 -> 37.3 mm, vias 0 -> 2
- net GPIO0: track 0.00 -> 36.9 mm
- net D+: track 0.00 -> 19.2 mm
- net D-: track 0.00 -> 18.9 mm
- net N$11: track 0.00 -> 10.2 mm
- net N$5: track 0.00 -> 9.48 mm
- net N$13: track 0.00 -> 9.09 mm
- net N$2: track 0.00 -> 4.72 mm
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
Commit message: programator zrobiony
Parts:
- moved R62 91.9 mm to (25.7, 58.7), turned to 90 degrees
- moved R61 81.2 mm to (21.4, 58.7), turned to 90 degrees
- moved R68 73.4 mm to (6.07, 61.5)
- moved R58 72.5 mm to (35.4, 20.2), turned to 180 degrees
- moved R66 68.2 mm to (11.6, 47.2), turned to 180 degrees
- moved T2 67.1 mm to (23.0, 63.7)
- moved R59 67.1 mm to (33.0, 38.5), turned to 90 degrees
- moved R67 67.0 mm to (6.04, 64.0)
- moved R60 65.9 mm to (11.4, 42.6)
- moved R64 65.6 mm to (23.5, 58.7), turned to 270 degrees
- moved R63 63.7 mm to (28.0, 58.7), turned to 270 degrees
- moved R65 62.6 mm to (11.5, 45.0), turned to 180 degrees
- moved T3 61.5 mm to (11.4, 52.3), turned to 180 degrees
- moved C3 54.2 mm to (41.6, 34.8), turned to 270 degrees
- moved R57 44.4 mm to (30.5, 38.4), turned to 270 degrees
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Routing:
- net GPIO0: track 36.9 -> 130.6 mm, vias 0 -> 4
- net RXD: track 38.4 -> 109.7 mm
- net TXD: track 37.3 -> 105.6 mm, vias 2 -> 4
- net +3V3: track 152.1 -> 213.0 mm, vias 4 -> 6
- net GPIO3: track 0.00 -> 43.6 mm, vias 0 -> 2
- net +5V: track 94.7 -> 136.6 mm
- net GPIO1: track 0.00 -> 31.6 mm
- net GPIO2: track 0.00 -> 25.9 mm, vias 0 -> 2
- net GND: track 103.5 -> 129.0 mm, vias 4 -> 6
- net LL2: track 0.00 -> 19.3 mm, vias 0 -> 2
- net RESET: track 39.0 -> 58.3 mm, vias 2 -> 4
- net SDA: track 0.00 -> 16.9 mm
- net LL1: track 0.00 -> 15.3 mm
- net N$19: track 0.00 -> 12.0 mm
- net ENABLE: track 0.00 -> 9.19 mm
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- added copper zone on layer 16, net GND
Other:
- board text added: "3,3V"
- board text added: "5V"
- board text added: "ANTENNA"
- board text added: "DTR"
- board text added: "ESP-01"
- board text added: "GND"
- board text added: "GPIO - ON"
- board text added: "GPIO0"
- board text added: "GPIO1"
- board text added: "GPIO2"
- board text added: "GPIO3"
- board text added: "RESET"
- board text added: "RTS"
- board text added: "RX"
- board text added: "TX"
- board text added: "USB - UART"
- board text added: "VCC"

Commit message: usb-uart skonczone, druga skonczona w 50%
Connections:
- net +3V3: now also J2.5; no longer J2.7
- net GND: now also J2.7; no longer J2.9
- net GPIO0: now also J2.9; no longer J2.10
- net GPIO1: now also S1.2; no longer S1.1
- net GPIO3: now also S1.1; no longer S1.2
- net RESET: now also J2.10
- net RXD: now also J2.4, U$1.RXD, U$4.A2; no longer J2.5, U$1.TXD, U$4.D1
- net TXD: now also J2.3, U$1.TXD, U$4.D1; no longer J2.4, U$1.RXD, U$4.A2
Routing:
- net GND: track 129.0 -> 155.3 mm
- net RXD: track 109.7 -> 88.3 mm
- net RESET: track 58.3 -> 70.7 mm
- net TXD: track 105.6 -> 94.1 mm
- net GPIO1: track 31.6 -> 41.6 mm
- net GPIO3: track 43.6 -> 47.8 mm
- net +3V3: track 213.0 -> 214.4 mm
- net GPIO0: track 130.6 -> 131.7 mm

Commit message: pierwsza docelowa wersja
Routing:
- net RESET: track 70.7 -> 48.9 mm
- net TXD: track 94.1 -> 86.0 mm
- net RXD: track 88.3 -> 80.3 mm
- net DTR: track 58.3 -> 53.9 mm
- net GND: track 155.3 -> 152.4 mm
Changed lines of the file:
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@@
 <layer number="47" name="Measures" color="7" fill="1" visible="no" active="yes"/>
 <layer number="48" name="Document" color="7" fill="1" visible="no" active="yes"/>
-<layer number="49" name="Reference" color="7" fill="1" visible="no" active="yes"/>
+<layer number="49" name="Reference" color="7" fill="1" visible="yes" active="yes"/>
 <layer number="50" name="dxf" color="7" fill="1" visible="no" active="no"/>
 <layer number="51" name="tDocu" color="7" fill="1" visible="yes" active="yes"/>
@@
 <layer number="99" name="SpiceOrder" color="7" fill="1" visible="no" active="no"/>
 <layer number="100" name="Muster" color="7" fill="1" visible="no" active="no"/>
-<layer number="101" name="Hidden" color="15" fill="1" visible="no" active="yes"/>
+<layer number="101" name="Hidden" color="15" fill="1" visible="yes" active="yes"/>
 <layer number="102" name="Changes" color="12" fill="1" visible="no" active="yes"/>
 <layer number="103" name="tMap" color="7" fill="1" visible="no" active="no"/>
@@
 <text x="20.75" y="64.75" size="1.778" layer="37" ratio="12">ANTENNA</text>
 <text x="20" y="56" size="2.7" layer="37" ratio="12">ESP-01</text>
-<text x="37" y="67" size="1.778" layer="37" ratio="12">GPIO - ON</text>
-<text x="1" y="63.125" size="1.778" layer="37" ratio="12">GPIO0</text>
-<text x="1" y="60.625" size="1.778" layer="37" ratio="12">GPIO1</text>
-<text x="1" y="58" size="1.778" layer="37" ratio="12">GPIO2</text>
-<text x="1" y="55.5" size="1.778" layer="37" ratio="12">GPIO3</text>
-<text x="19.625" y="30.125" size="1.6764" layer="37" font="vector" ratio="12" rot="R90">DTR</text>
-<text x="21.625" y="30.125" size="1.6764" layer="37" font="vector" ratio="12" rot="R90">RTS</text>
-<text x="23.5" y="30.125" size="1.6764" layer="37" font="vector" ratio="12" rot="R90">RESET</text>
-<text x="25.5" y="30.125" size="1.6764" layer="37" font="vector" ratio="12" rot="R90">GPIO0</text>
-<text x="29.75" y="30.125" size="1.6764" layer="37" font="vector" ratio="12" rot="R90">RX</text>
-<text x="27.625" y="30.125" size="1.6764" layer="37" font="vector" ratio="12" rot="R90">TX</text>
-<text x="31.625" y="30.125" size="1.6764" layer="37" font="vector" ratio="12" rot="R90">GND</text>
-<text x="33.625" y="30.125" size="1.6764" layer="37" font="vector" ratio="12" rot="R90">3,3V</text>
-<text x="2.375" y="1.625" size="2.1844" layer="37" ratio="12">3,3V</text>
-<text x="45.875" y="5.625" size="1.778" layer="37" ratio="12">3,3V</text>
-<text x="46" y="8" size="1.778" layer="37" ratio="12">VCC</text>
-<text x="46" y="10" size="1.778" layer="37" ratio="12">5V</text>
-<text x="17" y="21" size="2.54" layer="37" ratio="12">USB - UART</text>
+<text x="37" y="67" size="1.778" layer="49" ratio="12">GPIO - ON</text>
+<text x="1" y="63.125" size="1.778" layer="49" ratio="12">GPIO0</text>
+<text x="1" y="60.625" size="1.778" layer="49" ratio="12">GPIO1</text>
+<text x="1" y="58" size="1.778" layer="49" ratio="12">GPIO2</text>
+<text x="1" y="55.5" size="1.778" layer="49" ratio="12">GPIO3</text>
+<text x="19.625" y="30.125" size="1.6764" layer="49" font="vector" ratio="12" rot="R90">DTR</text>
+<text x="21.625" y="30.125" size="1.6764" layer="49" font="vector" ratio="12" rot="R90">RTS</text>
+<text x="23.5" y="30.125" size="1.6764" layer="49" font="vector" ratio="12" rot="R90">RESET</text>
+<text x="25.5" y="30.125" size="1.6764" layer="49" font="vector" ratio="12" rot="R90">GPIO0</text>
+<text x="29.75" y="30.125" size="1.6764" layer="49" font="vector" ratio="12" rot="R90">RX</text>
+<text x="27.625" y="30.125" size="1.6764" layer="49" font="vector" ratio="12" rot="R90">TX</text>
+<text x="31.625" y="30.125" size="1.6764" layer="49" font="vector" ratio="12" rot="R90">GND</text>
+<text x="33.625" y="30.125" size="1.6764" layer="49" font="vector" ratio="12" rot="R90">3,3V</text>
+<text x="2.375" y="1.625" size="2.1844" layer="49" ratio="12">3,3V</text>
+<text x="45.875" y="5.625" size="1.778" layer="49" ratio="12">3,3V</text>
+<text x="46" y="8" size="1.778" layer="49" ratio="12">VCC</text>
+<text x="46" y="10" size="1.778" layer="49" ratio="12">5V</text>
+<text x="17" y="21" size="2.54" layer="49" ratio="12">USB - UART</text>
 <text x="15.125" y="60.625" size="1.778" layer="37" ratio="12">TX</text>
 <text x="15" y="55.5" size="1.778" layer="37" ratio="12">RX</text>
+<wire x1="22.75" y1="23.5" x2="34.75" y2="23.5" width="0.8128" layer="101"/>
+<wire x1="18.75" y1="21.625" x2="18.875" y2="21.5" width="0.8128" layer="101"/>
+<wire x1="18.875" y1="21.5" x2="23" y2="21.5" width="0.8128" layer="101"/>
 </plain>
 <attributes>
@@
 <wire x1="30.75" y1="27.72" x2="30.75" y2="30.5" width="0.8128" layer="16"/>
 <via x="30.75" y="30.5" extent="1-16" drill="0.8" diameter="1.5"/>
-<wire x1="30.75" y1="30.5" x2="31" y2="30.5" width="0.8128" layer="1"/>
-<wire x1="32.75" y1="32.25" x2="31" y2="30.5" width="0.8128" layer="1"/>
-<wire x1="33" y1="32.25" x2="32.75" y2="32.25" width="0.8128" layer="1"/>
 <via x="33" y="32.25" extent="1-16" drill="0.8" diameter="1.5"/>
 <wire x1="33" y1="32.25" x2="33.03" y2="32.22" width="0.8128" layer="16"/>
@@
 <wire x1="33.625" y1="50.5" x2="33.625" y2="56.625" width="0.508" layer="1"/>
 <via x="33.625" y="56.625" extent="1-16" drill="0.8" diameter="1.5"/>
+<wire x1="49.12" y1="37.01" x2="49.12" y2="34.47" width="0" layer="19" extent="1-1"/>
+<wire x1="30.75" y1="30.5" x2="33" y2="32.25" width="0" layer="19" extent="1-1"/>
+<wire x1="20.35" y1="47.15" x2="22.4" y2="47.15" width="0" layer="19" extent="16-16"/>
+<wire x1="21.17" y1="10.27" x2="23.31" y2="10.41" width="0" layer="19" extent="16-16"/>
+<wire x1="18.96" y1="10.29" x2="21.17" y2="10.27" width="0" layer="19" extent="16-16"/>
 </signal>
 <signal name="TXD">
@@
 <wire x1="28.75" y1="27.72" x2="28.75" y2="30.5" width="0.8128" layer="16"/>
 <via x="28.75" y="30.5" extent="1-16" drill="0.8" diameter="1.5"/>
-<wire x1="28.75" y1="30.5" x2="28.5" y2="30.75" width="0.8128" layer="1"/>
-<wire x1="28.5" y1="38.5" x2="28.5" y2="30.75" width="0.8128" layer="1"/>
 <via x="28.5" y="38.5" extent="1-16" drill="0.8" diameter="1.5"/>
 <wire x1="28.5" y1="38.5" x2="28.5" y2="39" width="0.8128" layer="16"/>
@@
 <wire x1="33.5" y1="13" x2="37.32" y2="9.18" width="0.8128" layer="16"/>
 <wire x1="37.32" y1="9.18" x2="37.93" y2="9.18" width="0.8128" layer="16"/>
+<wire x1="28.75" y1="30.5" x2="28.5" y2="38.5" width="0" layer="19" extent="1-1"/>
 </signal>
 <signal name="RTS">
@@
 <wire x1="24.9" y1="21.5" x2="23" y2="21.5" width="0.8128" layer="16"/>
 <via x="23" y="21.5" extent="1-16" drill="0.8" diameter="1.5"/>
-<wire x1="23" y1="21.5" x2="19" y2="21.5" width="0.8128" layer="1"/>
-<wire x1="19" y1="21.5" x2="18.75" y2="21.75" width="0.8128" layer="1"/>
 <via x="18.75" y="21.75" extent="1-16" drill="0.8" diameter="1.5"/>
 <wire x1="18.75" y1="27.72" x2="18.75" y2="21.75" width="0.8128" layer="16"/>
@@
 <wire x1="38.75" y1="34.75" x2="38.25" y2="35.25" width="0.8128" layer="16"/>
 <wire x1="38.25" y1="35.25" x2="24" y2="35.25" width="0.8128" layer="16"/>
+<wire x1="18.75" y1="21.75" x2="23" y2="21.5" width="0" layer="19" extent="1-1"/>
 </signal>
 <signal name="N$1">
@@
 <wire x1="22.75" y1="27.72" x2="22.75" y2="23.4626" width="0.8128" layer="16"/>
 <via x="22.75" y="23.4626" extent="1-16" drill="0.8" diameter="1.5"/>
-<wire x1="22.75" y1="23.4626" x2="34.7126" y2="23.4626" width="0.8128" layer="1"/>
-<wire x1="34.7126" y1="23.4626" x2="34.75" y2="23.5" width="0.8128" layer="1"/>
 <via x="34.75" y="23.5" extent="1-16" drill="0.8" diameter="1.5"/>
 <wire x1="34.75" y1="23.5" x2="35.75" y2="23.5" width="0.8128" layer="16"/>
@@
 <wire x1="22.75" y1="29.75" x2="23.25" y2="30.25" width="0.8128" layer="16"/>
 <via x="23.25" y="30.25" extent="1-16" drill="0.8" diameter="1.5"/>
-<wire x1="23.25" y1="30.25" x2="23.25" y2="40" width="0.8128" layer="1"/>
 <via x="23.25" y="40" extent="1-16" drill="0.8" diameter="1.5"/>
 <wire x1="36.31" y1="20.25" x2="39.25" y2="20.25" width="0.8128" layer="16"/>
@@
 <wire x1="47.25" y1="29.25" x2="46.625" y2="28.625" width="0.508" layer="16"/>
 <wire x1="46.625" y1="28.625" x2="46.625" y2="19" width="0.508" layer="16"/>
-<wire x1="34.75" y1="23.5" x2="36" y2="23.5" width="0" layer="19" extent="16-16"/>
+<wire x1="23.25" y1="30.25" x2="23.25" y2="40" width="0" layer="19" extent="1-1"/>
+<wire x1="34.75" y1="23.5" x2="22.75" y2="23.4626" width="0" layer="19" extent="1-1"/>
+<wire x1="36" y1="23.5" x2="34.75" y2="23.5" width="0" layer="19" extent="16-16"/>
 </signal>
 <signal name="GPIO0">
@@
 <wire x1="26.75" y1="27.72" x2="26.75" y2="30.5" width="0.8128" layer="16"/>
 <via x="26.75" y="30.5" extent="1-16" drill="0.8" diameter="1.5"/>
-<wire x1="26.75" y1="30.5" x2="26.75" y2="38.5" width="0.8128" layer="1"/>
 <via x="26.75" y="38.5" extent="1-16" drill="0.8" diameter="1.5"/>
 <wire x1="26.75" y1="38.5" x2="21.75" y2="38.5" width="0.8128" layer="16"/>
@@
 <wire x1="32" y1="17" x2="26.875" y2="22.125" width="0.8128" layer="16"/>
 <wire x1="32" y1="12.195" x2="32" y2="17" width="0.8128" layer="16"/>
+<wire x1="26.75" y1="30.5" x2="26.75" y2="38.5" width="0" layer="19" extent="1-1"/>
 </signal>
 <signal name="N$5">

Commit message: powiekszonyy odstepy miedzy sciezkami
Parts:
- removed J4: 62000311121, Headers:62000311121
- removed J7: 62000811121, Headers:62000811121
- added JP3: (no value), pinhead:1X08
- added JP4: (no value), pinhead:1X03
Connections:
- net +3V3: now also JP3.1; no longer J7.8
- net DTR: now also JP3.8; no longer J7.1
- net GND: now also JP3.2; no longer J7.7
- net GPIO0: now also JP3.5; no longer J7.4
- net N$11: now also JP4.2; no longer J4.2
- net N$13: now also JP4.1; no longer J4.3
- net N$5: now also JP4.3; no longer J4.1
- net RESET: now also JP3.6; no longer J7.3
- net RTS: now also JP3.7; no longer J7.2
- net RXD: now also JP3.4; no longer J7.5
- net TXD: now also JP3.3; no longer J7.6
Routing:
- net GPIO0: track 131.7 -> 127.9 mm, vias 4 -> 6
- net GND: track 152.4 -> 154.5 mm, vias 6 -> 4
- net RESET: track 48.9 -> 47.5 mm
- net DTR: track 53.9 -> 54.7 mm
